File: D1(Motherboard)/ESP32-D0WDQ6-V3.kicad_sch (KiCad schematic)
At the start: 25 parts, among them U7 ESP32-D0WDQ6-V3, U8 AT25SF081-SSHD-X, Y1 Crystal_GND24

Commit message: Upload New Version from USB
Changed lines of the file:
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@@
   (symbol (lib_id "Device:R") (at 58.42 177.8 180) (unit 1)
     (in_bom yes) (on_board yes)
-    (property "Reference" "R12" (id 0) (at 58.42 179.07 90)
+    (property "Reference" "R12" (id 0) (at 58.42 180.34 90)
       (effects (font (size 1.27 1.27)) (justify right))
     )

Commit message: Added ESP32 Datasheets to recources, started cleaning up layout for esp32
Parts:
- U7: footprint Package_DFN_QFN:QFN-48-1EP_6x6mm_P0.4mm_EP4.2x4.2mm -> Package_DFN_QFN:QFN-48-1EP_6x6mm_P0.4mm_EP4.3x4.3mm
Changed lines of the file:
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@@
     (property "Reference" "U7" (id 0) (at 109.855 47.5955 0))
     (property "Value" "ESP32-D0WDQ6-V3" (id 1) (at 109.855 50.3706 0))
-    (property "Footprint" "Package_DFN_QFN:QFN-48-1EP_6x6mm_P0.4mm_EP4.2x4.2mm" (id 2) (at 115.57 86.995 0)
+    (property "Footprint" "Package_DFN_QFN:QFN-48-1EP_6x6mm_P0.4mm_EP4.3x4.3mm" (id 2) (at 115.57 86.995 0)
       (effects (font (size 1.27 1.27)) hide)
     )
