File: D1(Motherboard)/D1(Motherboard).kicad_sch (KiCad schematic)
At the start: 71 parts, among them J1 WR-FPC_0.5mm_ZIF_V, J2 USB_C_Receptacle_USB2.0, J3 B2B-PH-K-S, Q1 NX2301P.215, SW1 CHS-02A, U1 ESP32-S2, U2 ICM-20602, U3 WR-FPC_0.5mm_ZIF_H, U4 MIC5353-3.3YMT, U5 FAN5331SX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

Commit message: Potentially move over to ESP32-S2-MINI-1U
Parts:
- added U8: ESP32-S2-MINI-1, Espressif:ESP32-S2-MINI-1U, symbol Espressif:ESP32-S2-MINI-1
Other:
- note added: "MAYBE MOVE TO ESP32-S2-MINI-1U"
- note added: "https://docs.espressif.com/projects/esp-idf/en/latest/esp32s2/api-reference/peripherals/spi_master.html#overview-of-esp32-s2-s-spi-peripherals SPI2 HAS 6 CS PINS, THEN USE SPI3 FOR ICM20602"
Changed lines of the file:
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@@
     (effects (font (size 5 5) (thickness 1) bold italic) (justify left bottom))
   )
+  (text "MAYBE MOVE TO ESP32-S2-MINI-1U" (at 2.54 15.24 0)
+    (effects (font (size 5 5) (thickness 1) bold italic) (justify left bottom))
+  )
   (text "All Parts Aquired" (at 158.115 69.85 0)
     (effects (font (size 1.27 1.27)) (justify left bottom))
@@
     (effects (font (size 5 5) (thickness 1) bold italic) (justify left bottom))
   )
+  (text "https://docs.espressif.com/projects/esp-idf/en/latest/esp32s2/api-reference/peripherals/spi_master.html#overview-of-esp32-s2-s-spi-peripherals\n\nSPI2 HAS 6 CS PINS, THEN USE SPI3 FOR ICM20602\n\n"
+    (at 1.27 -3.81 0)
+    (effects (font (size 5 5) (thickness 1) bold italic) (justify left bottom))
+  )
   (global_label "VDD_SPI" (shape input) (at 270.51 165.1 90) (fields_autoplaced)
     (effects (font (size 1.27 1.27)) (justify left))
@@
     (pin "2")
   )
+  (symbol (lib_id "Espressif:ESP32-S2-MINI-1") (at 119.38 259.08 0) (unit 1)
+    (in_bom yes) (on_board yes) (fields_autoplaced)
+    (property "Reference" "U8" (id 0) (at 120.015 208.28 0))
+    (property "Value" "ESP32-S2-MINI-1" (id 1) (at 120.015 210.82 0))
+    (property "Footprint" "Espressif:ESP32-S2-MINI-1U" (id 2) (at 119.38 304.8 0)
+      (effects (font (size 1.27 1.27)) hide)
+    )
+    (property "Datasheet" "https://www.espressif.com/sites/default/files/documentation/esp32-s2-mini-1_esp32-s2-mini-1u_datasheet_en.pdf" (id 3) (at 118.11 259.08 0)
+      (effects (font (size 1.27 1.27)) hide)
+    )
+    (pin "43")
+    (pin "44")
+    (pin "45")
+    (pin "46")
+    (pin "1")
+    (pin "10")
+    (pin "11")
+    (pin "12")
+    (pin "13")
+    (pin "14")
+    (pin "15")
+    (pin "16")
+    (pin "17")
+    (pin "18")
+    (pin "19")
+    (pin "2")
+    (pin "20")
+    (pin "21")
+    (pin "22")
+    (pin "23")
+    (pin "24")
+    (pin "25")
+    (pin "26")
+    (pin "27")
+    (pin "28")
+    (pin "29")
+    (pin "3")
+    (pin "30")
+    (pin "31")
+    (pin "32")
+    (pin "33")
+    (pin "34")
+    (pin "35")
+    (pin "36")
+    (pin "37")
+    (pin "38")
+    (pin "39")
+    (pin "4")
+    (pin "40")
+    (pin "41")
+    (pin "42")
+    (pin "5")
+    (pin "6")
+    (pin "7")
+    (pin "8")
+    (pin "9")
+  )
   (symbol (lib_id "Device:L") (at 274.32 104.14 90) (unit 1)
     (in_bom yes) (on_board yes)
@@
       (reference "U7") (unit 1) (value "W25Q128JVS") (footprint "Package_SO:SOIC-8_5.23x5.23mm_P1.27mm")
     )
+    (path "/5f0f4914-432d-4e36-8115-2a8f3e154413"
+      (reference "U8") (unit 1) (value "ESP32-S2-MINI-1") (footprint "Espressif:ESP32-S2-MINI-1U")
+    )
     (path "/0c08d59a-87e7-4346-bbc7-d02a0356c794"

Commit message: Looking into moving to Mini Modulate and copying adafruit schematic
Parts:
- removed C22: 10u, Capacitor_SMD:C_0603_1608Metric, symbol Device:C
- removed C23: 1u, Capacitor_SMD:C_0603_1608Metric, symbol Device:C
- removed C24: 0.1u, Capacitor_SMD:C_0603_1608Metric, symbol Device:C
- removed C26: TBD, Capacitor_SMD:C_0603_1608Metric, symbol Device:C
- removed L2: 2n, Inductor_SMD:L_0603_1608Metric, symbol Device:L
- added C? (x2): 0.1u, Capacitor_SMD:C_0603_1608Metric, symbol Device:C
Connections:
- net +3V3: now also U8.3 (3V3), C?.1, C?.1
- net Boot: now also U8.4 (GPIO0/BOOT); no longer U1.5 (GPIO0/BOOT)
- net D+: now also U8.24 (USB_D+/ADC2_CH9/GPIO20); no longer U1.26 (GPIO20/ADC2_CH9/USB_D+)
- net D-: now also U8.23 (USB_D-/ADC2_CH8/GPIO19); no longer U1.25 (GPIO19/ADC2_CH8/USB_D-)
- net GND: now also U8.1 (GND), U8.2 (GND), U8.30 (GND), U8.42 (GND), U8.43 (GND), U8.46 (GND), C?.2, C?.2
- net Reset: now also U8.45 (CHIP/PU/RESET); no longer U1.56 (CHIP_PU/RESET)
- net U0RXD: now also U8.40 (GPIO44/U0RXD/PROG); no longer U1.49 (U0RXD/GPIO44)
- net at U1.48 (U0TXD/GPIO43): no longer R13.1
- net at U8.39 (GPIO43/U0TXD/PROG): now also R13.1
Other:
- note added: "LC709203 TO MONITOR BATTER AND BATTERY PERCENTAGE. IT CAN BE USED OVER I2C"
- note added: "https://shop.pimoroni.com/products/adafruit-esp32-s2-feather-2-mb-psram-and-stemma-qt-qwiic"
- moved on the sheet: R13, U8
