File: D1(Motherboard)/D1(Motherboard).kicad_pcb (KiCad board)
At the start: 4 copper layers, 38 x 35 mm, 51 parts, among them J1 WR-FPC_0.5mm_ZIF_V, J2 USB_C_Receptacle_USB2.0, J3 B2B-PH-K-S, Q1 NX2301P.215, SW1 CHS-02A, U1 ESP32-S2-MINI-1, U2 ICM-20602, U3 SSD1351, U4 MIC5353-3.3YMT, U5 FAN5331SX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

Commit message: Finished rough layout
Parts:
- moved C17 52.0 mm to (47.3, 46.3), turned to 180 degrees
- moved C15 51.1 mm to (45.0, 44.0)
- moved C16 51.1 mm to (48.8, 44.0)
- moved U4 51.1 mm to (46.9, 44.1)
- moved C12 48.2 mm to (39.4, 61.1), turned to -90 degrees
- moved SW1 44.3 mm to (36.3, 60.1), turned to 90 degrees
- moved C13 39.0 mm to (39.4, 58.0), turned to -90 degrees
- moved C14 21.5 mm to (69.8, 65.2), turned to 0 degrees
- moved R7 19.8 mm to (63.4, 61.6), turned to -90 degrees
- moved R8 19.3 mm to (66.4, 62.5)
- moved U5 19.2 mm to (69.3, 62.7)
- moved C19 18.4 mm to (64.9, 61.6), turned to 90 degrees
- moved D4 18.2 mm to (64.5, 57.7)
- moved L1 17.9 mm to (68.5, 58.1)
- moved C1 16.6 mm to (64.1, 63.8), turned to 180 degrees
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Connections:
- J1 pad 12: Display5_CS -> Display3_CS
- J1 pad 14: Display6_CS -> Display2_CS
- J1 pad 4: RST -> Reset
- J1 pad 6: Display2_CS -> Display6_CS
- J1 pad 8: Display3_CS -> Display5_CS
- U1 pad 11: Display1_CS -> Display6_CS
- U1 pad 12: Display2_CS -> Display5_CS
- U1 pad 13: Display3_CS -> Display4_CS
- U1 pad 14: Display4_CS -> Display3_CS
- U1 pad 15: Display5_CS -> Display2_CS
- U1 pad 16: Display6_CS -> Display1_CS
- U1 pad 8: INT -> unconnected-(U1-Pad8)
- U1 pad 9: RST -> INT
- U3 pad 21: RST -> Reset
Routing:
- net MOSI: track 8.40 -> 30.9 mm
- net D-: track 8.84 -> 26.3 mm, vias 2 -> 3
- net CLK: track 10.2 -> 27.3 mm
- net DC: track 0.00 -> 16.8 mm, vias 0 -> 1
- net Display1_CS: track 0.00 -> 12.8 mm
- net +5V: track 3.90 -> 11.2 mm, vias 0 -> 4
- net 13V: track 3.39 -> 10.6 mm
- net GND: track 25.3 -> 29.1 mm, vias 1 -> 0
- net Reset: track 0.50 -> 4.03 mm
- net D+: track 20.0 -> 22.5 mm
- net Net-(C8-Pad1): track 0.00 -> 1.96 mm
- net Net-(C7-Pad1): track 0.00 -> 1.69 mm
- net Net-(R5-Pad1): track 0.00 -> 1.60 mm
- net Display5_CS: track 17.3 -> 18.8 mm
- net INT: track 0.00 -> 1.26 mm, vias 0 -> 1
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- added copper zone on In1.Cu, net +5V

Commit message: More Layout
Routing:
- net Boot: track 0.00 -> 5.16 mm
- net Reset: track 4.03 -> 6.14 mm
Changed lines of the file:
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@@
   (segment (start 49.375 55.98) (end 49.375 57.385) (width 0.25) (layer "F.Cu") (net 33))
   (segment (start 49.235 55.84) (end 49.375 55.98) (width 0.25) (layer "F.Cu") (net 33))
-  (segment (start 38.695 57.499998) (end 38.695 57.995) (width 0.25) (layer "F.Cu") (net 36))
   (segment (start 68.685 33.965) (end 69.73 33.965) (width 0.4) (layer "F.Cu") (net 36))
+  (segment (start 36.89 57.575) (end 38.995 57.575) (width 0.25) (layer "F.Cu") (net 36))
   (segment (start 69.73 33.965) (end 70.485 34.72) (width 0.4) (layer "F.Cu") (net 36))
+  (segment (start 38.995 57.575) (end 39.35 57.22) (width 0.25) (layer "F.Cu") (net 36))
   (segment (start 70.485 34.72) (end 70.485 36.14) (width 0.4) (layer "F.Cu") (net 36))
+  (segment (start 35.62 58.08) (end 37.86 60.32) (width 0.25) (layer "F.Cu") (net 37))
+  (segment (start 35.62 57.575) (end 35.62 58.08) (width 0.25) (layer "F.Cu") (net 37))
+  (segment (start 37.86 60.32) (end 39.35 60.32) (width 0.25) (layer "F.Cu") (net 37))
   (segment (start 45.3375 43.315) (end 45.025 43.0025) (width 0.25) (layer "F.Cu") (net 39))
   (segment (start 70.59 65.195) (end 70.59 64.38) (width 0.4) (layer "F.Cu") (net 39))

Commit message: Test Commit
Parts:
- moved C15 23.6 mm to (21.7, 40.3)
- moved C16 23.6 mm to (25.5, 40.3)
- moved C17 23.6 mm to (24.1, 42.6)
- moved U4 23.6 mm to (23.6, 40.4)
Routing:
- net Net-(D3-Pad2): track 0.00 -> 4.85 mm
Changed lines of the file:
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@@
   )
   (footprint "Capacitor_SMD:C_0603_1608Metric" (layer "F.Cu")
-    (at 45.02 44.025 90)
+    (at 21.74 40.345 90)
     (descr "Capacitor SMD 0603 (1608 Metric), square (rectangular) end terminal, IPC_7351 nominal, (Body size source: IPC-SM-782 page 76, https://www.pcb-3d.com/wordpress/wp-content/uploads/ipc-sm-782a_amendment_1_and_2.pdf), generated with kicad-footprint-generator")
     (tags "capacitor")
@@
   )
   (footprint "Capacitor_SMD:C_0603_1608Metric" (layer "F.Cu")
-    (at 47.33 46.325 180)
+    (at 24.05 42.645 180)
     (descr "Capacitor SMD 0603 (1608 Metric), square (rectangular) end terminal, IPC_7351 nominal, (Body size source: IPC-SM-782 page 76, https://www.pcb-3d.com/wordpress/wp-content/uploads/ipc-sm-782a_amendment_1_and_2.pdf), generated with kicad-footprint-generator")
     (tags "capacitor")
@@
   )
   (footprint "Capacitor_SMD:C_0603_1608Metric" (layer "F.Cu")
-    (at 48.77 44.025 -90)
+    (at 25.49 40.345 -90)
     (descr "Capacitor SMD 0603 (1608 Metric), square (rectangular) end terminal, IPC_7351 nominal, (Body size source: IPC-SM-782 page 76, https://www.pcb-3d.com/wordpress/wp-content/uploads/ipc-sm-782a_amendment_1_and_2.pdf), generated with kicad-footprint-generator")
     (tags "capacitor")
@@
   )
   (footprint "Package_DFN_QFN:MLF-6-1EP_1.6x1.6mm_P0.5mm_EP0.5x1.26mm" (layer "F.Cu")
-    (at 46.9 44.115 -90)
+    (at 23.62 40.435 -90)
     (descr "MLF, 6 Pin (http://ww1.microchip.com/downloads/en/DeviceDoc/mic5353.pdf), generated with kicad-footprint-generator ipc_noLead_generator.py")
     (tags "MLF NoLead")
@@
   (segment (start 51.335 38.56) (end 52.835 38.56) (width 0.25) (layer "F.Cu") (net 5))
   (segment (start 58.375 56.085) (end 58.375 57.385) (width 0.25) (layer "F.Cu") (net 5))
-  (segment (start 46.9 43.315) (end 46.9 44.115) (width 0.25) (layer "F.Cu") (net 6))
-  (segment (start 45.705 44.115) (end 46.9 44.115) (width 0.4) (layer "F.Cu") (net 6))
+  (segment (start 23.62 39.635) (end 23.62 40.435) (width 0.25) (layer "F.Cu") (net 6))
+  (segment (start 22.425 40.435) (end 23.62 40.435) (width 0.4) (layer "F.Cu") (net 6))
   (segment (start 68.75596 62.685) (end 68.1375 62.685) (width 0.4) (layer "F.Cu") (net 6))
-  (segment (start 45.02 44.8) (end 45.705 44.115) (width 0.4) (layer "F.Cu") (net 6))
+  (segment (start 21.74 41.12) (end 22.425 40.435) (width 0.4) (layer "F.Cu") (net 6))
   (segment (start 68.17952 64.33452) (end 65.40952 64.33452) (width 0.4) (layer "F.Cu") (net 6))
   (segment (start 46.375 58.209022) (end 46.324511 58.259511) (width 0.25) (layer "F.Cu") (net 6))
@@
   (segment (start 69.35048 63.27952) (end 68.75596 62.685) (width 0.4) (layer "F.Cu") (net 6))
   (segment (start 40.1075 39.885) (end 38.72 39.885) (width 0.25) (layer "F.Cu") (net 6))
-  (segment (start 48.77 43.25) (end 47.905 44.115) (width 0.4) (layer "F.Cu") (net 6))
+  (segment (start 25.49 39.57) (end 24.625 40.435) (width 0.4) (layer "F.Cu") (net 6))
   (segment (start 67.95 52.8175) (end 67.95 53.625) (width 0.25) (layer "F.Cu") (net 6))
   (segment (start 45.375 58.209022) (end 45.375 57.385) (width 0.25) (layer "F.Cu") (net 6))
@@
   (segment (start 66.6 61.65) (end 67.635 62.685) (width 0.4) (layer "F.Cu") (net 6))
   (segment (start 46.375 57.385) (end 46.375 58.209022) (width 0.25) (layer "F.Cu") (net 6))
-  (segment (start 47.905 44.115) (end 46.9 44.115) (width 0.4) (layer "F.Cu") (net 6))
+  (segment (start 24.625 40.435) (end 23.62 40.435) (width 0.4) (layer "F.Cu") (net 6))
   (segment (start 38.72 39.885) (end 38.39 39.555) (width 0.25) (layer "F.Cu") (net 6))
   (segment (start 69.04 65.195) (end 68.17952 64.33452) (width 0.4) (layer "F.Cu") (net 6))
@@
   (segment (start 35.62 57.575) (end 35.62 58.08) (width 0.25) (layer "F.Cu") (net 37))
   (segment (start 37.86 60.32) (end 39.35 60.32) (width 0.25) (layer "F.Cu") (net 37))
-  (segment (start 45.3375 43.315) (end 45.025 43.0025) (width 0.25) (layer "F.Cu") (net 39))
+  (segment (start 22.0575 39.635) (end 21.745 39.3225) (width 0.25) (layer "F.Cu") (net 39))
   (segment (start 70.59 65.195) (end 70.59 64.38) (width 0.4) (layer "F.Cu") (net 39))
-  (segment (start 45.02 43.25) (end 46.335 43.25) (width 0.2) (layer "F.Cu") (net 39))
-  (segment (start 47.19048 42.66548) (end 46.60952 42.66548) (width 0.2) (layer "F.Cu") (net 39))
+  (segment (start 21.74 39.57) (end 23.055 39.57) (width 0.2) (layer "F.Cu") (net 39))
+  (segment (start 23.91048 38.98548) (end 23.32952 38.98548) (width 0.2) (layer "F.Cu") (net 39))
   (segment (start 70.59 63.8125) (end 70.4125 63.635) (width 0.4) (layer "F.Cu") (net 39))
-  (segment (start 47.4 42.875) (end 47.19048 42.66548) (width 0.2) (layer "F.Cu") (net 39))
-  (segment (start 47.4 43.315) (end 47.4 42.875) (width 0.2) (layer "F.Cu") (net 39))
-  (segment (start 46.60952 42.66548) (end 46.4 42.875) (width 0.2) (layer "F.Cu") (net 39))
+  (segment (start 24.12 39.195) (end 23.91048 38.98548) (width 0.2) (layer "F.Cu") (net 39))
+  (segment (start 24.12 39.635) (end 24.12 39.195) (width 0.2) (layer "F.Cu") (net 39))
+  (segment (start 23.32952 38.98548) (end 23.12 39.195) (width 0.2) (layer "F.Cu") (net 39))
   (segment (start 70.4125 63.635) (end 70.4125 62.6575) (width 0.4) (layer "F.Cu") (net 39))
-  (segment (start 46.4 42.875) (end 46.4 43.315) (width 0.2) (layer "F.Cu") (net 39))
+  (segment (start 23.12 39.195) (end 23.12 39.635) (width 0.2) (layer "F.Cu") (net 39))
   (segment (start 70.06 61.3825) (end 70.4125 61.735) (width 0.4) (layer "F.Cu") (net 39))
   (segment (start 70.4125 62.6575) (end 70.4125 61.735) (width 0.4) (layer "F.Cu") (net 39))
   (segment (start 70.59 64.38) (end 70.59 63.8125) (width 0.4) (layer "F.Cu") (net 39))
   (segment (start 70.06 58.135) (end 70.06 61.3825) (width 0.4) (layer "F.Cu") (net 39))
-  (segment (start 46.335 43.25) (end 46.4 43.315) (width 0.2) (layer "F.Cu") (net 39))
+  (segment (start 23.055 39.57) (end 23.12 39.635) (width 0.2) (layer "F.Cu") (net 39))
   (via (at 39.905 35.775) (size 0.8) (drill 0.4) (layers "F.Cu" "B.Cu") (free) (net 39))
   (via (at 39.875 34.405) (size 0.8) (drill 0.4) (layers "F.Cu" "B.Cu") (free) (net 39))
   (via (at 70.4125 62.6575) (size 0.8) (drill 0.4) (layers "F.Cu" "B.Cu") (net 39))
   (via (at 70.59 64.38) (size 0.8) (drill 0.4) (layers "F.Cu" "B.Cu") (net 39))
-  (segment (start 48.5875 44.915) (end 48.775 44.7275) (width 0.25) (layer "F.Cu") (net 40))
-  (segment (start 48.655 44.915) (end 48.77 44.8) (width 0.2) (layer "F.Cu") (net 40))
-  (segment (start 47.4 44.915) (end 48.655 44.915) (width 0.2) (layer "F.Cu") (net 40))
+  (segment (start 25.3075 41.235) (end 25.495 41.0475) (width 0.25) (layer "F.Cu") (net 40))
+  (segment (start 25.375 41.235) (end 25.49 41.12) (width 0.2) (layer "F.Cu") (net 40))
+  (segment (start 24.12 41.235) (end 25.375 41.235) (width 0.2) (layer "F.Cu") (net 40))
   (segment (start 63.385 62.39) (end 64.905 62.39) (width 0.4) (layer "F.Cu") (net 41))
   (segment (start 66.445 63.3) (end 66.11 63.3) (width 0.4) (layer "F.Cu") (net 41))
@@
   (segment (start 67.28 63.3) (end 66.445 63.3) (width 0.4) (layer "F.Cu") (net 41))
   (segment (start 64.905 62.39) (end 64.925 62.37) (width 0.4) (layer "F.Cu") (net 41))
+  (segment (start 43.0825 42.435) (end 44.1725 41.345) (width 0.25) (layer "F.Cu") (net 42))
+  (segment (start 46.18 41.345) (end 47.1 40.425) (width 0.25) (layer "F.Cu") (net 42))
+  (segment (start 44.1725 41.345) (end 46.18 41.345) (width 0.25) (layer "F.Cu") (net 42))
   (segment (start 41.5075 42.435) (end 41.25952 42.18702) (width 0.25) (layer "F.Cu") (net 43))
   (segment (start 40.635 38.935) (end 40.1075 38.935) (width 0.25) (layer "F.Cu") (net 43))

Commit message: Almost finished alyout and added links to look at
Parts:
- moved C15 24.3 mm to (44.8, 47.8), turned to 180 degrees
- moved C17 23.5 mm to (47.1, 47.1), turned to 90 degrees
- moved U4 22.0 mm to (44.9, 46.0), turned to 0 degrees
- moved C16 19.7 mm to (44.8, 44.1), turned to 0 degrees
Routing:
- net +3V3: track 11.0 -> 22.2 mm
- net Display6_CS: track 19.2 -> 20.4 mm
- net Display5_CS: track 18.8 -> 19.9 mm
- net Display4_CS: track 18.7 -> 19.7 mm
- net Display3_CS: track 18.6 -> 19.5 mm
- net Display2_CS: track 17.6 -> 18.3 mm
- net GND: track 29.1 -> 29.8 mm, vias 0 -> 1
- net +5V: vias 4 -> 7
